Commit message: restructured xacro file

File: prbt_robot_support/urdf/prbt.xacro (robot description, xacro)
@@ -10,10 +10,8 @@
     <xacro:include filename="$(find prbt_robot_support)/urdf/prbt.ros2_control.xacro" />
     <!-- instantiate the robot -->
-    <xacro:prbt prefix="$(arg robot_prefix)" />
     <link name="world"/>
-    <joint name="world-base_link-fixed" type="fixed">
-        <parent link="world"/>
-        <child link="$(arg robot_prefix)base_link"/>
-    </joint>
+    <xacro:prbt prefix="$(arg robot_prefix)" parent="world">
+        <origin xyz="0 0 0" rpy="0 0 0" />
+    </xacro:prbt>
     <xacro:prbt_ros2_control
         name="$(arg robot_prefix)"

File: prbt_robot_support/urdf/prbt_macro.xacro (robot description, xacro)
@@ -1,5 +1,5 @@
 <?xml version="1.0"?>
 <robot xmlns:xacro="http://www.ros.org/wiki/xacro">
-  <xacro:macro name="prbt" params="prefix">
+  <xacro:macro name="prbt" params="prefix parent *origin">
     <!-- Height of Foot -->
     <xacro:property name="L0" value="0.2604" />
@@ -10,4 +10,9 @@
     <!-- Distance last joint to flange -->
     <xacro:property name="L3" value="0.0840" />
+    <joint name="${prefix}base_link_${parent}_joint" type="fixed">
+      <xacro:insert_block name="origin" />
+      <parent link="${parent}"/>
+      <child link="${prefix}base_link"/>
+    </joint>
     <!-- robot foot link -->
     <link name="${prefix}base_link">

Commit message: remove ros2 control and sim related tags

File: prbt_robot_support/urdf/prbt.xacro (robot description, xacro)
@@ -1,5 +1,5 @@
 <?xml version="1.0"?>
 <robot xmlns:xacro="http://www.ros.org/wiki/xacro" name="prbt">
-    <xacro:arg name="robot_prefix" default="prbt_"/>
+    <xacro:arg name="robot_prefix" default=""/>
     <xacro:arg name="bus_config" default="$(find prbt_robot_support)/config/prbt/bus.yml"/>
     <xacro:arg name="master_config" default="$(find prbt_robot_support)/config/prbt/master.dcf"/>
@@ -14,10 +14,3 @@
         <origin xyz="0 0 0" rpy="0 0 0" />
     </xacro:prbt>
-    <xacro:prbt_ros2_control
-        name="$(arg robot_prefix)"
-        prefix="$(arg robot_prefix)"
-        bus_config="$(arg bus_config)"
-        master_config="$(arg master_config)"
-        can_interface_name="$(arg can_interface_name)"
-        master_bin="$(arg master_bin)" />
 </robot>

File: prbt_robot_support/urdf/prbt_macro.xacro (robot description, xacro)
@@ -90,5 +90,5 @@
         <inertia ixx="3.58e-2" ixy="0" ixz="0" iyy="3.22e-3" iyz="-1.45e-3" izz="3.66e-2" />
       </inertial>
-      <visual name="first">
+      <visual>
         <origin xyz="0 0 0" rpy="0 0 0" />
         <geometry>
@@ -278,114 +278,4 @@
       <child link="${prefix}tool0" />
     </joint>
-    <!-- transmissions for gazebo -->
-    <transmission name="${prefix}joint_1_trans">
-      <type>transmission_interface/SimpleTransmission</type>
-      <joint name="${prefix}joint_1">
-        <hardwareInterface>hardware_interface/PositionJointInterface</hardwareInterface>
-      </joint>
-      <actuator name="${prefix}joint_1_motor"/>
-    </transmission>
-    <transmission name="${prefix}joint_2_trans">
-      <type>transmission_interface/SimpleTransmission</type>
-      <joint name="${prefix}joint_2">
-        <hardwareInterface>hardware_interface/PositionJointInterface</hardwareInterface>
-      </joint>
-      <actuator name="${prefix}joint_2_motor"/>
-    </transmission>
-    <transmission name="${prefix}joint_3_trans">
-      <type>transmission_interface/SimpleTransmission</type>
-      <joint name="${prefix}joint_3">
-        <hardwareInterface>hardware_interface/PositionJointInterface</hardwareInterface>
-      </joint>
-      <actuator name="${prefix}joint_3_motor"/>
-    </transmission>
-    <transmission name="${prefix}joint_4_trans">
-      <type>transmission_interface/SimpleTransmission</type>
-      <joint name="${prefix}joint_4">
-        <hardwareInterface>hardware_interface/PositionJointInterface</hardwareInterface>
-      </joint>
-      <actuator name="${prefix}joint_4_motor"/>
-    </transmission>
-    <transmission name="${prefix}joint_5_trans">
-      <type>transmission_interface/SimpleTransmission</type>
-      <joint name="${prefix}joint_5">
-        <hardwareInterface>hardware_interface/PositionJointInterface</hardwareInterface>
-      </joint>
-      <actuator name="${prefix}joint_5_motor"/>
-    </transmission>
-    <transmission name="${prefix}joint_6_trans">
-      <type>transmission_interface/SimpleTransmission</type>
-      <joint name="${prefix}joint_6">
-        <hardwareInterface>hardware_interface/PositionJointInterface</hardwareInterface>
-      </joint>
-      <actuator name="${prefix}joint_6_motor"/>
-    </transmission>
-    <gazebo>
-      <plugin name="gazebo_ros_control" filename="libgazebo_ros_control.so">
-        <robotNamespace>prbt</robotNamespace>
-        <robotSimType>gazebo_ros_control/DefaultRobotHWSim</robotSimType>
-        <legacyModeNS>false</legacyModeNS>        <!-- Only used from ros-kinetic-gazebo-ros-control 2.5.18 -->
-      </plugin>
-    </gazebo>
-    <gazebo reference="${prefix}joint_1">
-      <provideFeedback>true</provideFeedback>
-    </gazebo>
-    <gazebo>
-      <plugin name="ft_sensor" filename="libgazebo_ros_ft_sensor.so">
-        <updateRate>100.0</updateRate>
-        <topicName>prbt/ft_sensor/joint_1</topicName>
-        <jointName>${prefix}joint_1</jointName>
-      </plugin>
-    </gazebo>
-    <gazebo reference="${prefix}joint_2">
-      <provideFeedback>true</provideFeedback>
-    </gazebo>
-    <gazebo>
-      <plugin name="ft_sensor" filename="libgazebo_ros_ft_sensor.so">
-        <updateRate>100.0</updateRate>
-        <topicName>prbt/ft_sensor/joint_2</topicName>
-        <jointName>${prefix}joint_2</jointName>
-      </plugin>
-    </gazebo>
-    <gazebo reference="${prefix}joint_3">
-      <provideFeedback>true</provideFeedback>
-    </gazebo>
-    <gazebo>
-      <plugin name="ft_sensor" filename="libgazebo_ros_ft_sensor.so">
-        <updateRate>100.0</updateRate>
-        <topicName>prbt/ft_sensor/joint_3</topicName>
-        <jointName>${prefix}joint_3</jointName>
-      </plugin>
-    </gazebo>
-    <gazebo reference="${prefix}joint_4">
-      <provideFeedback>true</provideFeedback>
-    </gazebo>
-    <gazebo>
-      <plugin name="ft_sensor" filename="libgazebo_ros_ft_sensor.so">
-        <updateRate>100.0</updateRate>
-        <topicName>prbt/ft_sensor/joint_4</topicName>
-        <jointName>${prefix}joint_4</jointName>
-      </plugin>
-    </gazebo>
-    <gazebo reference="${prefix}joint_5">
-      <provideFeedback>true</provideFeedback>
-    </gazebo>
-    <gazebo>
-      <plugin name="ft_sensor" filename="libgazebo_ros_ft_sensor.so">
-        <updateRate>100.0</updateRate>
-        <topicName>prbt/ft_sensor/joint_5</topicName>
-        <jointName>${prefix}joint_5</jointName>
-      </plugin>
-    </gazebo>
-    <gazebo reference="${prefix}joint_6">
-      <provideFeedback>true</provideFeedback>
-    </gazebo>
-    <gazebo>
-      <plugin name="ft_sensor" filename="libgazebo_ros_ft_sensor.so">
-        <updateRate>100.0</updateRate>
-        <topicName>prbt/ft_sensor/joint_6</topicName>
-        <jointName>${prefix}joint_6</jointName>
-      </plugin>
-    </gazebo>
   </xacro:macro>
 </robot>
