Commit message: update file paths for gz

File: prbt_robot_support/urdf/prbt_macro.xacro (robot description, xacro)
@@ -24,5 +24,5 @@
         <origin xyz="0 0 0" rpy="0 0 0" />
         <geometry>
-          <mesh filename="package://prbt_robot_support/meshes/foot.dae" />
+          <mesh filename="file://$(find prbt_robot_support)/meshes/foot.dae" />
         </geometry>
       </visual>
@@ -53,5 +53,5 @@
         <origin xyz="0 0 0" rpy="0 0 0" />
         <geometry>
-          <mesh filename="package://prbt_robot_support/meshes/link_1.dae" />
+          <mesh filename="file://$(find prbt_robot_support)/meshes/link_1.dae" />
         </geometry>
       </visual>
@@ -93,5 +93,5 @@
         <origin xyz="0 0 0" rpy="0 0 0" />
         <geometry>
-          <mesh filename="package://prbt_robot_support/meshes/link_2.dae" />
+          <mesh filename="file://$(find prbt_robot_support)/meshes/link_2.dae" />
         </geometry>
       </visual>
@@ -127,5 +127,5 @@
         <origin xyz="0 0 0" rpy="0 0 0" />
         <geometry>
-          <mesh filename="package://prbt_robot_support/meshes/link_3.dae" />
+          <mesh filename="file://$(find prbt_robot_support)/meshes/link_3.dae" />
         </geometry>
       </visual>
@@ -167,5 +167,5 @@
         <origin xyz="0 0 0" rpy="0 0 0" />
         <geometry>
-          <mesh filename="package://prbt_robot_support/meshes/link_4.dae" />
+          <mesh filename="file://$(find prbt_robot_support)/meshes/link_4.dae" />
         </geometry>
       </visual>
@@ -201,5 +201,5 @@
         <origin xyz="0 0 0" rpy="0 0 0" />
         <geometry>
-          <mesh filename="package://prbt_robot_support/meshes/link_5.dae"/>
+          <mesh filename="file://$(find prbt_robot_support)/meshes/link_5.dae"/>
         </geometry>
       </visual>
@@ -249,10 +249,10 @@
         <mass value="0.02" />
         <origin xyz="0 0 0" />
-        <inertia ixx="0" ixy="0" ixz="0" iyy="0" iyz="0" izz="0" />
-      </inertial>
-      <visual>
-        <origin xyz="0 0 0" rpy="0 0 0" />
-        <geometry>
-          <mesh filename="package://prbt_robot_support/meshes/flange.dae"/>
+        <inertia ixx="0.001" ixy="0" ixz="0" iyy="0.001" iyz="0" izz="0.001" />
+      </inertial>
+      <visual>
+        <origin xyz="0 0 0" rpy="0 0 0" />
+        <geometry>
+          <mesh filename="file://$(find prbt_robot_support)/meshes/flange.dae"/>
         </geometry>
       </visual>
@@ -321,9 +321,9 @@
       <actuator name="${prefix}joint_6_motor"/>
     </transmission>
-    <gazebo>
+    <!-- <gazebo>
       <plugin name="gazebo_ros2_control" filename="libgazebo_ros2_control.so">
         <robotNamespace>prbt</robotNamespace>
         <robotSimType>gazebo_ros2_control/DefaultRobotHWSim</robotSimType>
-        <legacyModeNS>false</legacyModeNS>        <!-- Only used from ros-kinetic-gazebo-ros-control 2.5.18 -->
+        <legacyModeNS>false</legacyModeNS>
       </plugin>
     </gazebo>
@@ -387,5 +387,5 @@
         <jointName>${prefix}joint_6</jointName>
       </plugin>
-    </gazebo>
+    </gazebo> -->
   </xacro:macro>
 </robot>

Commit message: update path

File: prbt_robot_support/urdf/prbt_macro.xacro (robot description, xacro)
@@ -24,5 +24,5 @@
         <origin xyz="0 0 0" rpy="0 0 0" />
         <geometry>
-          <mesh filename="package://prbt_robot_support/meshes/foot.dae" />
+          <mesh filename="file://$(find prbt_robot_support)/meshes/foot.dae" />
         </geometry>
       </visual>
@@ -53,5 +53,5 @@
         <origin xyz="0 0 0" rpy="0 0 0" />
         <geometry>
-          <mesh filename="package://prbt_robot_support/meshes/link_1.dae" />
+          <mesh filename="file://$(find prbt_robot_support)/meshes/link_1.dae" />
         </geometry>
       </visual>
@@ -93,5 +93,5 @@
         <origin xyz="0 0 0" rpy="0 0 0" />
         <geometry>
-          <mesh filename="package://prbt_robot_support/meshes/link_2.dae" />
+          <mesh filename="file://$(find prbt_robot_support)/meshes/link_2.dae" />
         </geometry>
       </visual>
@@ -127,5 +127,5 @@
         <origin xyz="0 0 0" rpy="0 0 0" />
         <geometry>
-          <mesh filename="package://prbt_robot_support/meshes/link_3.dae" />
+          <mesh filename="file://$(find prbt_robot_support)/meshes/link_3.dae" />
         </geometry>
       </visual>
@@ -167,5 +167,5 @@
         <origin xyz="0 0 0" rpy="0 0 0" />
         <geometry>
-          <mesh filename="package://prbt_robot_support/meshes/link_4.dae" />
+          <mesh filename="file://$(find prbt_robot_support)/meshes/link_4.dae" />
         </geometry>
       </visual>
@@ -201,5 +201,5 @@
         <origin xyz="0 0 0" rpy="0 0 0" />
         <geometry>
-          <mesh filename="package://prbt_robot_support/meshes/link_5.dae"/>
+          <mesh filename="file://$(find prbt_robot_support)/meshes/link_5.dae"/>
         </geometry>
       </visual>
@@ -254,5 +254,5 @@
         <origin xyz="0 0 0" rpy="0 0 0" />
         <geometry>
-          <mesh filename="package://prbt_robot_support/meshes/flange.dae"/>
+          <mesh filename="file://$(find prbt_robot_support)/meshes/flange.dae"/>
         </geometry>
       </visual>

Commit message: fix inertia

File: prbt_robot_support/urdf/prbt_macro.xacro (robot description, xacro)
@@ -249,5 +249,5 @@
         <mass value="0.02" />
         <origin xyz="0 0 0" />
-        <inertia ixx="0" ixy="0" ixz="0" iyy="0" iyz="0" izz="0" />
+        <inertia ixx="0.001" ixy="0" ixz="0" iyy="0.001" iyz="0" izz="0.001" />
       </inertial>
       <visual>
